File: hw/USB-Mux.kicad_pcb (KiCad board)
At the start: 6 copper layers, 60 x 70 mm, 107 parts, among them J101 USB-61400416121, J102 USB-676432911, J103 USB-61400416121, J104 USB-676432911, J201 Conn_01x08, J202 Molex-105017-0001, J203 Conn_01x03, J204 Conn_01x02, J205 Conn_01x02, J206 Conn_01x02, J207 Conn_01x02, P201 Current-Probe, Q101 DTC114EE, Q102 DTC114EE, Q103 DTC114EE, Q104 DTC114EE, Q201 DTC114EE, U101 TS3USB3000, U102 TS3USB3000, U103 TPS22976, U104 TPS22976, U105 TUSB212, U201 STM32F401XX-LQFP64, U202 TLV62150A, X101 Lightpipe-5x12.7mm-Dome, X102 Lightpipe-5x12.7mm-Dome, X103 Lightpipe-5x12.7mm-Dome, X104 Lightpipe-5x12.7mm-Dome, X105 Lightpipe-5x12.7mm-Dome, X201 Mounting-Hole-M3, X202 Mounting-Hole-M3, X203 Mounting-Hole-M3, X204 Mounting-Hole-M3, Y201 MCSJK-7I-8.00-18-30-60-B-30

Commit message: Mark dnp components in schematic.
Other:
- board text added: "PCB Stack-Up: Top Layer: 35 um 2x Prepreg 2116: 230 um Inner Layer 1: 35 um Core: 300 um Inner Layer 2: 35 um 3x Prepreg 2116: 340um Inner Layer 3: 35 um Core: 300 um Inner Layer 4: 35 um 2x Prepreg 2116: 230um Bottom Layer: 35 um εr_FR4 = 4.6 USB-Trace: width = 180 um spacing = 100 um gnd_spacing = 200 um Zdiff = 93.584 Ω Zcomm = 43.745 Ω"
- board text removed: "PCB Stack-Up: Top Layer: 35 um 2x Prepreg 2116: 230 um Inner Layer 1: 35 um Core: 300 um Inner Layer 2: 35 um 3x Prepreg 2116: 340um Inner Layer 3: 35 um Core: 300 um Inner Layer 4: 35 um 2x Prepreg 2116: 230um Bottom Layer: 35 um εr_FR4 = 4.3 εr_soldermask = 3.2 USB-Trace: width = 180 um spacing = 100 um gnd_spacing = 200 um Zdiff = 93.584 Ω Zcomm = 43.745 Ω"
Changed lines of the file:
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@@
     (effects (font (size 1 1) (thickness 0.15)))
   )
-  (gr_text "PCB Stack-Up:\n\nTop Layer: 35 um\n2x Prepreg 2116: 230 um\nInner Layer 1: 35 um\nCore: 300 um\nInner Layer 2: 35 um\n3x Prepreg 2116: 340um\nInner Layer 3: 35 um\nCore: 300 um\nInner Layer 4: 35 um\n2x Prepreg 2116: 230um\nBottom Layer: 35 um\n\nεr_FR4 = 4.3\nεr_soldermask = 3.2\n\nUSB-Trace:\nwidth = 180 um\nspacing = 100 um\ngnd_spacing = 200 um\nZdiff = 93.584 Ω\nZcomm = 43.745 Ω" (at 155.2 36.6) (layer "Eco1.User")
+  (gr_text "PCB Stack-Up:\n\nTop Layer: 35 um\n2x Prepreg 2116: 230 um\nInner Layer 1: 35 um\nCore: 300 um\nInner Layer 2: 35 um\n3x Prepreg 2116: 340um\nInner Layer 3: 35 um\nCore: 300 um\nInner Layer 4: 35 um\n2x Prepreg 2116: 230um\nBottom Layer: 35 um\n\nεr_FR4 = 4.6\n\nUSB-Trace:\nwidth = 180 um\nspacing = 100 um\ngnd_spacing = 200 um\nZdiff = 93.584 Ω\nZcomm = 43.745 Ω" (at 155.2 36.6) (layer "Eco1.User")
     (effects (font (size 1 1) (thickness 0.15)) (justify left))
   )
